File: esp8266_pcb/gondola.brd (EAGLE design)
At the start: 75 x 42 mm, 22 parts, among them X1 1751248, X2 1751264

Commit message: some work on pcb
Parts:
- R6: value 10k -> 100k
- moved U$3 4.64 mm to (48.0, 18.7), turned to 90 degrees
- moved R6 2.13 mm to (62.4, 16.5), turned to 180 degrees
- moved C1 1.33 mm to (63.3, 20.4), turned to 0 degrees
- moved R7 0.99 mm to (62.5, 23.7)
Connections:
- net +12V: now also U$3.VIN; no longer U$3.1
- net +5V: now also U$3.VOUT; no longer U$3.3
- net GND: now also U$3.GND; no longer U$3.2
Routing:
- net +3V3: track 53.2 -> 41.9 mm
- net GND: track 122.9 -> 127.5 mm, vias 1 -> 0
- net +12V: track 40.1 -> 43.0 mm
- net +5V: track 35.6 -> 32.7 mm
- net M_EN: track 11.8 -> 13.6 mm
- net MS3: track 13.5 -> 12.1 mm
- net 2A: track 26.8 -> 25.4 mm
- net 12V_IN: track 19.2 -> 18.4 mm
Other:
- board text added: "marvin.sieverding@tuhh.de"
- board text removed: "Marvin Sieverding"
