File: esp8266_pcb/gondola.sch (EAGLE design)
At the start: 22 parts, among them X1 1751248, X2 1751264

Commit message: some work on pcb
Parts:
- R6: value 10k -> 100k
Other:
- moved on the sheet: U$3
Changed lines of the file:
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@@
 <setting verticaltext="up"/>
 </settings>
-<grid distance="0.1" unitdist="inch" unit="inch" style="lines" multiple="1" display="yes" altdistance="0.01" altunitdist="inch" altunit="inch"/>
+<grid distance="0.1" unitdist="inch" unit="inch" style="lines" multiple="1" display="no" altdistance="0.01" altunitdist="inch" altunit="inch"/>
 <layers>
 <layer number="1" name="Top" color="4" fill="1" visible="no" active="no"/>
@@
 <part name="R7" library="adafruit" deviceset="R-US_" device="R0805" value="100k"/>
 <part name="GND5" library="supply1" library_urn="urn:adsk.eagle:library:371" deviceset="GND" device=""/>
-<part name="R6" library="adafruit" deviceset="R-US_" device="R0805" value="10k"/>
+<part name="R6" library="adafruit" deviceset="R-US_" device="R0805" value="100k"/>
 <part name="+3V2" library="supply1" library_urn="urn:adsk.eagle:library:371" deviceset="+3V3" device=""/>
 <part name="C1" library="adafruit" deviceset="CPOL-US" device="153CLV-0605" value="100µF"/>
@@
 <instance part="U$3" gate="G$1" x="66.04" y="-104.14"/>
 <instance part="P+3" gate="1" x="53.34" y="-83.82"/>
-<instance part="P+4" gate="1" x="-27.94" y="35.56"/>
+<instance part="P+4" gate="1" x="-27.94" y="45.72"/>
 <instance part="GND6" gate="1" x="5.08" y="2.54"/>
 <instance part="LED3_5V" gate="G$1" x="119.38" y="-114.3"/>
@@
 <segment>
 <pinref part="P+4" gate="1" pin="+5V"/>
-<wire x1="-27.94" y1="33.02" x2="-27.94" y2="17.78" width="0.1524" layer="91"/>
+<wire x1="-27.94" y1="43.18" x2="-27.94" y2="17.78" width="0.1524" layer="91"/>
 <pinref part="U$2" gate="G$1" pin="VBAT"/>
 <wire x1="-27.94" y1="17.78" x2="12.7" y2="17.78" width="0.1524" layer="91"/>
